File: hardware/mainmodule/JLCPCB.kicad_pcb (KiCad board)
At the start: 2 copper layers, 83.8 x 61 mm, 74 parts, among them J1 USB+, J10 Conn_01x04, J2 To LED_MOD_0, J3 To EXT_MOD_1, J4 V24_IN, J5 Temp, J6 Presence, J7 Neo, J8 AUX, J9 Conn_01x04, Q1 Si3456DDV, Q2 Si3456DDV, Q3 Si3456DDV, Q4 Si3456DDV, Q5 Si3456DDV, Q6 Si3456DDV, SW1 SW_Push, SW2 SW_Push, U1 ESP32-C6-WROOM-1, U2 VEML6040A3OG, U3 74HCT244, U4 DS18B20, U5 MC34063AD

Commit message: Update version in Silkscreen.
Other:
- board text added: "Main Module v1.1"
- board text removed: "Main Module v1"
