File: hardware/mainmodule/JLCPCB.kicad_sch (KiCad schematic)
At the start: 63 parts, among them J1 USB+, J10 Conn_01x04, J2 To LED_MOD_0, J3 To EXT_MOD_1, J4 V24_IN, J5 Temp, J6 Presence, J7 Neo, J8 AUX, J9 Conn_01x04, Q1 Si3456DDV, Q2 Si3456DDV, Q3 Si3456DDV, Q4 Si3456DDV, Q5 Si3456DDV, Q6 Si3456DDV, SW1 SW_Push, SW2 SW_Push, U1 ESP32-C6-WROOM-1, U3 74HCT244, U4 DS18B20, U5 MC34063AD

Commit message: Apply open hardware licenses.
Other:
- title: Beste Lampe Main Module -> besteLampe! LED Main Moudule
Changed lines of the file:
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@@
   (paper "USLetter")
   (title_block
-    (title "Beste Lampe Main Module")
+		(title "besteLampe! LED Main Moudule")
     (date "2024-01-07")
-    (rev "1")
-    (comment 1 "Design for JLCPCB 1-2 Layer Service")
-  )
+		(rev "1.0")
+		(comment 1 "See  https://lenaschimmel.de/besteLampe! for the source and more information")
+		(comment 2 "This source describes Open Hardware and is licensed under the CERN-OHL-S v2.")
+		(comment 3 "Copyright 2024 Lena Schimmel <mail@lenaschimmel.de>")
+    (comment 4 "Design for JLCPCB 1-2 Layer Service")
+	)
   (junction (at 27.305 34.925) (diameter 0) (color 0 0 0 0)
   )
