File: hardware/ledmodule/LED_Module_A/LED_Module_A.kicad_sch (KiCad schematic)
At the start: 147 parts, among them J2 Connector Header Surface Moun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, U1 DS18B20U+

Commit message: Apply open hardware licenses.
Other:
- title: (none) -> besteLampe! LED Moudule A
Changed lines of the file:
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@@
 (kicad_sch (version 20230121) (generator eeschema)
   (paper "A4")
+  (title_block
+		(title "besteLampe! LED Moudule A")
+		(date "2024-02-19")
+		(rev "1.0")
+		(comment 1 "See  https://lenaschimmel.de/besteLampe! for the source and more information")
+		(comment 2 "This source describes Open Hardware and is licensed under the CERN-OHL-S v2.")
+		(comment 3 "Copyright 2024 Lena Schimmel <mail@lenaschimmel.de>")
+	)
   (junction (at 22.86 100.33) (diameter 0) (color 0 0 0 0)
   )
