File: hardware/ledmodule/LED_Test_Module/LED_Test_Module.kicad_sch (KiCad schematic)
At the start: 0 parts

Commit message: Apply open hardware licenses.
Other:
- title: (none) -> LED Test Moudule
Changed lines of the file:
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@@
 (kicad_sch (version 20230121) (generator eeschema)
   (paper "A4")
+  (title_block
+		(title "LED Test Moudule")
+		(date "2024-03-02")
+		(rev "1.0")
+		(comment 1 "See  https://lenaschimmel.de/besteLampe! for the source and more information")
+		(comment 2 "This source describes Open Hardware and is licensed under the CERN-OHL-S v2.")
+		(comment 3 "Copyright 2024 Lena Schimmel <mail@lenaschimmel.de>")
+	)
   (sheet_instances
     (path "/" (page "1"))
