File: hardware/ledmodule/LED_Module_A_Adaptor/LED_Module_A_Adaptor.kicad_sch (KiCad schematic)
At the start: 7 parts, among them J1 Conn_LED_Board, J2 Conn_Cable, J3 Conn_01x04, J4 Conn_01x02

Commit message: Fix / add meta data in title_block for all LED modules.
Other:
- title: (none) -> besteLampe! LED Module A Adaptor
Changed lines of the file:
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@@
 	(paper "A4")
 	(title_block
+		(title "besteLampe! LED Module A Adaptor")
 		(date "2024-04-22")
 		(rev "v2")
+		(comment 1 "See  https://lenaschimmel.de/besteLampe! for the source and more information")
+		(comment 2 "This source describes Open Hardware and is licensed under the CERN-OHL-S v2.")
+		(comment 3 "Copyright 2024 Lena Schimmel <mail@lenaschimmel.de>")
 	)
 	(junction
