File: hardware/ledmodule/LED_Module_B/LED_Module_B.kicad_sch (KiCad schematic)
At the start: 32 parts, among them J1 Conn_01x10, J2 Conn_01x10

Commit message: Fix / add meta data in title_block for all LED modules.
Other:
- title: (none) -> besteLampe! LED Module B
Changed lines of the file:
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@@
 (kicad_sch (version 20230121) (generator eeschema)
   (paper "A4")
+  (title_block
+		(title "besteLampe! LED Module B")
+		(date "2024-03-16")
+		(rev "1.0")
+		(comment 1 "See  https://lenaschimmel.de/besteLampe! for the source and more information")
+		(comment 2 "This source describes Open Hardware and is licensed under the CERN-OHL-S v2.")
+		(comment 3 "Copyright 2024 Lena Schimmel <mail@lenaschimmel.de>")
+	)
   (wire (pts (xy 35.56 44.45) (xy 35.56 80.645))
     (stroke (width 0) (type default))
