File: hardware/ledmodule/LED_Module_D/LED_Module_D.kicad_sch (KiCad schematic)
At the start: 62 parts, among them J1 Conn_01x10_Pin, J2 Conn_01x02_Pin, Q1 Si3456DDV, Q10 Si3456DDV, Q2 Si3456DDV, Q3 Si3456DDV, Q4 Si3456DDV, Q5 Si3456DDV, Q6 Si3456DDV, Q7 Si3456DDV, Q8 Si3456DDV, Q9 Si3456DDV, U1 TMP1075DGK, U2 74HCT244, U3 24AA02-OT

Commit message: Fix / add meta data in title_block for all LED modules.
Other:
- title: (none) -> besteLampe! LED Module D
Changed lines of the file:
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@@
 	(generator_version "8.0")
 	(paper "A4")
+	(title_block
+		(title "besteLampe! LED Module D")
+		(date "2024-05-05")
+		(rev "1.1")
+		(comment 1 "See  https://lenaschimmel.de/besteLampe! for the source and more information")
+		(comment 2 "This source describes Open Hardware and is licensed under the CERN-OHL-S v2.")
+		(comment 3 "Copyright 2024 Lena Schimmel <mail@lenaschimmel.de>")
+	)
 	(junction
 		(at 85.09 88.9)
