File: hardware/abl/sensor_adapter/sensor_adapter.kicad_pcb (KiCad board)
At the start: 4 copper layers, 59.4 x 44.1 mm, 10 parts, among them J1 Conn_02x05_Odd_Even, J2 Conn_02x05_Odd_Even, J3 Conn_02x05_Odd_Even

Commit message: Many small adjustments for the next production run.
Other:
- outline, holes or cut-outs redrawn
Changed lines of the file:
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@@
-			)
-			(layer "dielectric 1"
-				(type "core")
-				(thickness 1.51)
-				(material "FR4")
-				(epsilon_r 4.5)
-				(loss_tangent 0.02)
-			)
-			(layer "B.Cu"
-				(type "copper")
-				(thickness 0.035)
-			)
-			(layer "B.Mask"
-				(type "Bottom Solder Mask")
-				(thickness 0.01)
-			)
-			(layer "B.Paste"
-				(type "Bottom Solder Paste")
-			)
-			(layer "B.SilkS"
-				(type "Bottom Silk Screen")
-			)
-			(layer "F.SilkS"
-				(type "Top Silk Screen")
-				(color "Black")
-			)
-			(layer "F.Paste"
-				(type "Top Solder Paste")
-			)
-			(layer "F.Mask"
-				(type "Top Solder Mask")
-				(color "White")
-				(thickness 0.01)
-			)
-			(layer "F.Cu"
-				(type "copper")
-				(thickness 0.035)
 			)
 			(layer "dielectric 1"
@@
 			(layer "B.Mask"
 				(type "Bottom Solder Mask")
-				(color "White")
 				(thickness 0.01)
 			)
@@
 			(layer "B.SilkS"
 				(type "Bottom Silk Screen")
-				(color "Black")
 			)
 			(copper_finish "HAL lead-free")
@@
 	)
 	(gr_line
-		(start 92 42.39375)
+		(start 92 40.282843)
 		(end 92 44.09375)
 		(stroke
@@
 	)
 	(gr_line
-		(start 114 47.49375)
-		(end 118 47.49375)
+		(start 113.6 47.49375)
+		(end 118.4 47.49375)
 		(stroke
 			(width 0.05)
@@
 	)
 	(gr_arc
-		(start 119 46.49375)
-		(mid 118.707107 47.200857)
-		(end 118 47.49375)
+		(start 119.4 46.49375)
+		(mid 119.107124 47.200889)
+		(end 118.4 47.49375)
 		(stroke
 			(width 0.05)
@@
 	)
 	(gr_arc
-		(start 119 45.49375)
-		(mid 119.292893 44.786643)
-		(end 120 44.49375)
+		(start 119.4 45.49375)
+		(mid 119.692876 44.786611)
+		(end 120.4 44.49375)
 		(stroke
 			(width 0.05)
@@
 	(gr_line
 		(start 110.8 44.49375)
-		(end 112 44.49375)
+		(end 111.6 44.49375)
 		(stroke
 			(width 0.05)
@@
 	)
 	(gr_line
-		(start 113 45.49375)
-		(end 113 46.49375)
+		(start 112.6 45.49375)
+		(end 112.6 46.49375)
 		(stroke
 			(width 0.05)
@@
 	)
 	(gr_line
-		(start 120 44.49375)
+		(start 120.4 44.49375)
 		(end 124.221616 44.49375)
 		(stroke
@@
 	)
 	(gr_arc
-		(start 114 47.49375)
-		(mid 113.292893 47.200857)
-		(end 113 46.49375)
+		(start 113.6 47.49375)
+		(mid 112.892911 47.200854)
+		(end 112.6 46.49375)
 		(stroke
 			(width 0.05)
@@
 	)
 	(gr_line
-		(start 119 46.49375)
-		(end 119 45.49375)
+		(start 119.4 46.49375)
+		(end 119.4 45.49375)
 		(stroke
 			(width 0.05)
@@
 	)
 	(gr_arc
-		(start 92 42.39375)
-		(mid 92.117157 42.110907)
-		(end 92.4 41.99375)
+		(start 92 40.282843)
+		(mid 92.11714 39.999968)
+		(end 92.4 39.882843)
 		(stroke
 			(width 0.05)
@@
 	(gr_line
 		(start 95.3 44.09375)
-		(end 95.3 42.39375)
+		(end 95.3 40.282843)
 		(stroke
 			(width 0.05)
@@
 	)
 	(gr_arc
-		(start 94.9 41.99375)
-		(mid 95.182843 42.110907)
-		(end 95.3 42.39375)
+		(start 94.9 39.882843)
+		(mid 95.182825 40.000003)
+		(end 95.3 40.282843)
 		(stroke
 			(width 0.05)
@@
 	)
 	(gr_arc
-		(start 112 44.49375)
-		(mid 112.707107 44.786643)
-		(end 113 45.49375)
+		(start 111.6 44.49375)
+		(mid 112.307089 44.786646)
+		(end 112.6 45.49375)
 		(stroke
 			(width 0.05)
@@
 	)
 	(gr_line
-		(start 94.9 41.99375)
-		(end 92.4 41.99375)
-		(stroke
-			(width 0.05)
+		(start 94.9 39.882843)
+		(end 92.4 39.882843)
+		(stroke
+			(width 0.05)
