File: hardware/abl/Feather C6/Adafruit Feather ESP32-C6.kicad_sch (KiCad schematic)
At the start: 45 parts, among them J1 Conn_01x10_Pin, J2 Conn_01x10_Pin, Q3 DMG3415U, SW1 KMR2, SW2 KMR2, U1 ESP32-C6-MINI_MINI, U2 AP2112/RT9080-3.3, U3 MCP73831T-2ACI/OT, U4 AHT20-F, U5 AP2112/RT9080-3.3, X1 JSTPH, X2 MAX17048/T, X3 USB C

Commit message: WIP feature conf (does not compile)
Parts:
- removed C12: 10uF, Adafruit Feather ESP32-C6:_0805MP, symbol Adafruit Feather ESP32-C6-eagle-import:CAP_CERAMIC_0805MP
- removed CHG0: ORANGE, Adafruit Feather ESP32-C6:CHIPLED_0603_NOOUTLINE, symbol Adafruit Feather ESP32-C6-eagle-import:LED0603_NOOUTLINE
- removed CONN1: JST SH, Adafruit Feather ESP32-C6:JST_SH4_RA, symbol Adafruit Feather ESP32-C6-eagle-import:STEMMA_I2C_QTRA
- removed LED1: WS2812B_3535FULL, Adafruit Feather ESP32-C6:LED3535_FULLPADS, symbol Adafruit Feather ESP32-C6-eagle-import:WS2812B_3535FULL
- removed R2, R4: 5.1K, Adafruit Feather ESP32-C6:0603-NO, symbol Adafruit Feather ESP32-C6-eagle-import:RESISTOR_0603_NOOUT
- removed unit 1 of R3
- removed unit 2 of R3
- removed SJ1: SOLDERJUMPERCLOSED, Adafruit Feather ESP32-C6:SOLDERJUMPER_CLOSEDWIRE, symbol Adafruit Feather ESP32-C6-eagle-import:SOLDERJUMPERCLOSED
- removed U$34, U$35: FIDUCIAL_1MM, Adafruit Feather ESP32-C6:FIDUCIAL_1MM, symbol Adafruit Feather ESP32-C6-eagle-import:FIDUCIAL_1MM
- removed U3: MCP73831T-2ACI/OT, Adafruit Feather ESP32-C6:SOT23-5, symbol Adafruit Feather ESP32-C6-eagle-import:MCP73831/2
- removed X1: JSTPH, Adafruit Feather ESP32-C6:JSTPH2_BATT, symbol Adafruit Feather ESP32-C6-eagle-import:CON_JST_PH_2PIN_MT_BATT
- removed X2: MAX17048/T, Adafruit Feather ESP32-C6:TDFN8_2X2MM, symbol Adafruit Feather ESP32-C6-eagle-import:MAX17048/T
- C1, C2, C6, C7, C8, C9: footprint Adafruit Feather ESP32-C6:0805-NO -> Capacitor_SMD:C_0805_2012Metric; LCSC Part # (none) -> C15850
- C10, C4: footprint Adafruit Feather ESP32-C6:0603-NO -> Capacitor_SMD:C_0603_1608Metric; LCSC Part # (none) -> C15849
- C11, R3, U4, U5: now not fitted; now left out of the parts list
- D3: LCSC Part # (none) -> C7207730
- D4: LCSC Part # (none) -> C122863
- J1, J2: LCSC Part # (none) -> C2905418
- JP1: LCSC Part # (none) -> C2905421
- JP3: LCSC Part # (none) -> C2905419
- Q3: LCSC Part # (none) -> C7202986
- R1, R10, R5, R8: footprint Adafruit Feather ESP32-C6:0603-NO -> Resistor_SMD:R_0603_1608Metric; LCSC Part # (none) -> C23186
- R12, R6, R7: footprint Adafruit Feather ESP32-C6:0603-NO -> Resistor_SMD:R_0603_1608Metric; LCSC Part # (none) -> C25803
- SW1, SW2: LCSC Part # (none) -> C221676
- U$31, U$32: now not fitted
- U1: LCSC Part # (none) -> C5736265
- U2: LCSC Part # (none) -> C51118
- X3: LCSC Part # (none) -> C2927039
Other:
- note removed: "1.0K = 1000mA"
- note removed: "10K = 100mA"
- note removed: "2.0K = 500mA"
- note removed: "5.0K = 200mA"
- note removed: "LIPO CHARGING"
- note removed: "NEOPIXEL"
