File: hardware/abl/Feather C6/Adafruit Feather ESP32-C6.kicad_sch (KiCad schematic)
At the start: 35 parts, among them J1 Conn_01x10_Pin, J2 Conn_01x10_Pin, Q3 DMG3415U, SW1 KMR2, SW2 KMR2, U1 ESP32-C6-MINI_MINI, U2 AP2112/RT9080-3.3, U4 AHT20-F, U5 AP2112/RT9080-3.3, X3 USB C

Commit message: Update to KiCad 9, ready for prodution.
Other:
- company: (none) -> besteLampe!
- title: (none) -> ESP32-C6 Feather
Changed lines of the file:
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@@
 (kicad_sch
-	(version 20231120)
+	(version 20250114)
 	(generator "eeschema")
-	(generator_version "8.0")
+	(generator_version "9.0")
 	(paper "User" 425.45 298.602)
+	(title_block
+		(title "ESP32-C6 Feather")
+		(date "2025-01-05")
+		(rev "v1.1")
+		(company "besteLampe!")
+		(comment 1 "See  https://beste-lampe.de for the source and more information")
+		(comment 2 "This source describes Open Hardware and is licensed under the CERN-OHL-S v2.")
+		(comment 3 "Copyright 2025 Lena Schimmel <mail@lenaschimmel.de>")
+		(comment 4 "Based on ESP32-C6 Feather STEMMA QT by Adafruit")
+	)
+	(text "RESET"
+		(exclude_from_sim no)
+		(at 50.8 116.84 90)
+		(effects
+			(font
+				(size 1.778 1.5113)
+			)
+			(justify left bottom)
+		)
+	)
+	(text "POWER AND FILTERING"
+		(exclude_from_sim no)
+		(at 165.1 40.64 0)
+		(effects
+			(font
+				(size 1.778 1.5113)
+			)
+			(justify left bottom)
+		)
+	)
+	(text "LED"
+		(exclude_from_sim no)
+		(at 144.78 111.76 0)
+		(effects
+			(font
+				(size 1.778 1.5113)
+			)
+			(justify left bottom)
+		)
+	)
 	(junction
 		(at 335.28 193.04)
@@
 		)
 	)
-	(text "RESET"
-		(exclude_from_sim no)
-		(at 50.8 116.84 90)
-		(effects
-			(font
-				(size 1.778 1.5113)
-			)
-			(justify left bottom)
-		)
-	)
-	(text "POWER AND FILTERING"
-		(exclude_from_sim no)
-		(at 165.1 40.64 0)
-		(effects
-			(font
-				(size 1.778 1.5113)
-			)
-			(justify left bottom)
-		)
-	)
-	(text "LED"
-		(exclude_from_sim no)
-		(at 144.78 111.76 0)
-		(effects
-			(font
-				(size 1.778 1.5113)
-			)
-			(justify left bottom)
-		)
-	)
 	(label "SCL"
 		(at 340.36 205.74 0)
-		(fields_autoplaced yes)
 		(effects
 			(font
@@
 	(label "SDA"
 		(at 106.68 190.5 0)
-		(fields_autoplaced yes)
 		(effects
 			(font
@@
 	(label "MISO"
 		(at 200.66 203.2 0)
-		(fields_autoplaced yes)
 		(effects
 			(font
@@
 	(label "A0"
 		(at 35.56 180.34 0)
-		(fields_autoplaced yes)
 		(effects
 			(font
@@
 	(label "IO8"
 		(at 144.78 193.04 0)
-		(fields_autoplaced yes)
 		(effects
 			(font
@@
 	(label "D+"
 		(at 68.58 45.72 0)
-		(fields_autoplaced yes)
 		(effects
 			(font
@@
 	(label "MOSI"
 		(at 106.68 198.12 0)
-		(fields_autoplaced yes)
 		(effects
 			(font
@@
 	(label "VSENSOR"
 		(at 358.14 185.42 0)
-		(fields_autoplaced yes)
 		(effects
 			(font
@@
 	(label "IO7"
 		(at 35.56 195.58 0)
-		(fields_autoplaced yes)
 		(effects
 			(font
@@
 	(label "EN"
 		(at 160.02 66.04 0)
-		(fields_autoplaced yes)
 		(effects
 			(font
@@
 	(label "IO15"
 		(at 144.78 185.42 0)
-		(fields_autoplaced yes)
 		(effects
 			(font
@@
 	(label "SCL"
 		(at 106.68 187.96 0)
-		(fields_autoplaced yes)
 		(effects
 			(font
@@
 	(label "I2C_PWR"
 		(at 266.7 203.2 0)
-		(fields_autoplaced yes)
 		(effects
 			(font
@@
 	(label "A5"
 		(at 200.66 195.58 0)
-		(fields_autoplaced yes)
 		(effects
 			(font
@@
 	(label "EN"
 		(at 144.78 180.34 0)
-		(fields_autoplaced yes)
 		(effects
 			(font
@@
 	(label "VHI"
 		(at 276.86 200.66 0)
-		(fields_autoplaced yes)
 		(effects
 			(font
@@
 	(label "A4"
 		(at 200.66 193.04 0)
-		(fields_autoplaced yes)
 		(effects
 			(font
@@
 	(label "SDA"
 		(at 144.78 205.74 0)
-		(fields_autoplaced yes)
 		(effects
 			(font
@@
 	(label "IO14"
 		(at 106.68 177.8 0)
-		(fields_autoplaced yes)
 		(effects
 			(font
@@
 	(label "A2/IO6"
 		(at 144.78 198.12 0)
-		(fields_autoplaced yes)
 		(effects
 			(font
@@
 	(label "TX"
 		(at 109.22 167.64 0)
-		(fields_autoplaced yes)
 		(effects
 			(font
@@
 	(label "A4"
 		(at 35.56 185.42 0)
-		(fields_autoplaced yes)
 		(effects
 			(font
@@
 	(label "A3/IO5"
 		(at 144.78 200.66 0)
-		(fields_autoplaced yes)
 		(effects
 			(font
@@
 	(label "A2/IO6"
 		(at 200.66 187.96 0)
-		(fields_autoplaced yes)
 		(effects
 			(font
@@
 	(label "A5"
 		(at 35.56 182.88 0)
-		(fields_autoplaced yes)
 		(effects
 			(font
@@
 	(label "IO7"
 		(at 144.78 195.58 0)
-		(fields_autoplaced yes)
 		(effects
 			(font
@@
 	(label "IO9/BOOT/NEOPIX"
 		(at 27.94 200.66 0)
-		(fields_autoplaced yes)
 		(effects
 			(font
@@
 	(label "IO14"
 		(at 144.78 187.96 0)
-		(fields_autoplaced yes)
 		(effects
 			(font
@@
 	(label "IO15"
 		(at 106.68 180.34 0)
-		(fields_autoplaced yes)
 		(effects
 			(font
@@
 	(label "IO9/BOOT/NEOPIX"
 		(at 101.6 121.92 0)
-		(fields_autoplaced yes)
 		(effects
 			(font
@@
 	(label "RESET"
 		(at 38.1 162.56 0)
-		(fields_autoplaced yes)
 		(effects
 			(font
@@
 	(label "RX"
 		(at 109.22 170.18 0)
-		(fields_autoplaced yes)
 		(effects
 			(font
@@
 	(label "D-"
 		(at 68.58 48.26 0)
-		(fields_autoplaced yes)
 		(effects
 			(font
@@
 	(label "VHI"
 		(at 147.32 55.88 0)
-		(fields_autoplaced yes)
 		(effects
 			(font
@@
 	(label "SCK"
 		(at 200.66 198.12 0)
-		(fields_autoplaced yes)
 		(effects
 			(font
@@
 	(label "MISO"
 		(at 106.68 200.66 0)
-		(fields_autoplaced yes)
 		(effects
 			(font
@@
 	(label "TX"
 		(at 200.66 208.28 0)
-		(fields_autoplaced yes)
 		(effects
 			(font
@@
 	(label "IO0"
 		(at 144.78 190.5 0)
-		(fields_autoplaced yes)
 		(effects
 			(font
@@
 	(label "SCL"
 		(at 144.78 203.2 0)
-		(fields_autoplaced yes)
 		(effects
 			(font
@@
 	(label "IO0"
 		(at 35.56 175.26 0)
-		(fields_autoplaced yes)
 		(effects
 			(font
@@
 	(label "RESET"
 		(at 208.28 172.72 0)
-		(fields_autoplaced yes)
 		(effects
 			(font
@@
 	(label "RESET"
 		(at 60.96 124.46 0)
-		(fields_autoplaced yes)
 		(effects
 			(font
@@
 	(label "D-"
 		(at 35.56 208.28 0)
-		(fields_autoplaced yes)
 		(effects
 			(font
@@
 	(label "D+"
 		(at 35.56 210.82 0)
-		(fields_autoplaced yes)
 		(effects
 			(font
@@
 	(label "A3/IO5"
 		(at 35.56 190.5 0)
-		(fields_autoplaced yes)
 		(effects
 			(font
@@
 	(label "MOSI"
 		(at 200.66 200.66 0)
-		(fields_autoplaced yes)
 		(effects
 			(font
@@
 	(label "IO15"
 		(at 132.08 121.92 0)
-		(fields_autoplaced yes)
 		(effects
 			(font
@@
 	(label "SCK"
 		(at 106.68 195.58 0)
-		(fields_autoplaced yes)
 		(effects
 			(font
@@
 	(label "A1"
 		(at 35.56 187.96 0)
-		(fields_autoplaced yes)
 		(effects
 			(font
@@
 	(label "A3/IO5"
 		(at 200.66 190.5 0)
-		(fields_autoplaced yes)
 		(effects
 			(font
@@
 	(label "A0"
 		(at 200.66 182.88 0)
-		(fields_autoplaced yes)
 		(effects
 			(font
@@
 	(label "RX"
 		(at 200.66 205.74 0)
-		(fields_autoplaced yes)
 		(effects
 			(font
@@
 	(label "SDA"
 		(at 340.36 208.28 0)
-		(fields_autoplaced yes)
 		(effects
 			(font
@@
 	(label "A2/IO6"
 		(at 35.56 193.04 0)
-		(fields_autoplaced yes)
 		(effects
 			(font
@@
 	(label "A1"
 		(at 200.66 185.42 0)
-		(fields_autoplaced yes)
 		(effects
 			(font
@@
 	(label "IO9/BOOT/NEOPIX"
 		(at 200.66 210.82 0)
-		(fields_autoplaced yes)
 		(effects
 			(font
@@
 	(label "I2C_PWR"
 		(at 106.68 193.04 0)
-		(fields_autoplaced yes)
 		(effects
 			(font
@@
 	(label "IO8"
 		(at 35.56 198.12 0)
-		(fields_autoplaced yes)
 		(effects
 			(font
@@
 		)
 	)
+	(embedded_fonts no)
 )
