File: hardware/abl/controller/Feather_Ground.kicad_pcb (KiCad board)
At the start: 2 copper layers, 51.9 x 29.5 mm, 3 parts, among them J6 Conn_01x10_Pin, J7 Conn_01x10_Pin

Commit message: Fix missing ground collection - this PCB had *one* job!
Connections:
- A1 pad : (no net) -> GND
Other:
- board text added: "v1.1"
- board text removed: "v1.0"
Changed lines of the file:
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@@
 			(layers "*.Cu" "*.Mask")
 			(remove_unused_layers no)
+			(net 1 "GND")
 		)
 		(pad "" np_thru_hole oval
@@
 		(layer "Edge.Cuts")
 	)
-	(gr_text "v1.0"
-		(at 99.568 99.822 -0)
+	(gr_text "v1.1"
+		(at 99.568 99.822 0)
 		(layer "B.SilkS")
 		(effects
@@
 			(justify left bottom mirror)
 		)
-		(render_cache "v1.0" -0
+		(render_cache "v1.1" 0
 			(polygon
 				(pts
@@
 			(polygon
 				(pts
-					(xy 96.950017 98.639965) (xy 97.008347 98.647635) (xy 97.053998 98.658818) (xy 97.108901 98.680779)
-					(xy 97.151025 98.706029) (xy 97.194289 98.742853) (xy 97.196666 98.745294) (xy 97.231784 98.78919)
-					(xy 97.259734 98.838633) (xy 97.271075 98.864546) (xy 97.289072 98.917806) (xy 97.302146 98.972893)
-					(xy 97.303062 98.977727) (xy 97.311218 99.034011) (xy 97.315579 99.090132) (xy 97.317033 99.150971)
-					(xy 97.317001 99.160312) (xy 97.315014 99.222876) (xy 97.309936 99.280494) (xy 97.300346 99.340286)
-					(xy 97.284732 99.39983) (xy 97.282672 99.405935) (xy 97.259477 99.462704) (xy 97.231565 99.511682)
-					(xy 97.195412 99.556561) (xy 97.165692 99.583595) (xy 97.116569 99.615984) (xy 97.061995 99.638577)
-					(xy 97.012918 99.651168) (xy 96.956272 99.659631) (xy 96.896838 99.662452) (xy 96.841748 99.660038)
-					(xy 96.784064 99.651807) (xy 96.729434 99.637735) (xy 96.692024 99.62334) (xy 96.640979 99.593584)
-					(xy 96.596016 99.554033) (xy 96.592528 99.55029) (xy 96.557281 99.504093) (xy 96.530191 99.454089)
-					(xy 96.50782 99.396459) (xy 96.50585 99.39025) (xy 96.490934 99.330124) (xy 96.481928 99.270261)
-					(xy 96.477332 99.212928) (xy 96.475807 99.151252) (xy 96.693762 99.151252) (xy 96.695865 99.208838)
-					(xy 96.700912 99.26485) (xy 96.711738 99.325116) (xy 96.726601 99.373284) (xy 96.754994 99.425671)
-					(xy 96.76916 99.441716) (xy 96.818191 99.471735) (xy 96.838815 99.47703) (xy 96.895152 99.482689)
-					(xy 96.946272 99.478757) (xy 96.99346 99.462466) (xy 97.035311 99.427918) (xy 97.042391 99.418978)
-					(xy 97.068736 99.368371) (xy 97.078945 99.335651) (xy 97.090363 99.27849) (xy 97.092207 99.264889)
-					(xy 97.09693 99.208024) (xy 97.098228 99.151252) (xy 97.098212 99.144275) (xy 97.096582 99.08553)
-					(xy 97.091645 99.028806) (xy 97.081375 98.972613) (xy 97.064233 98.92074) (xy 97.035873 98.872058)
-					(xy 97.021162 98.856434) (xy 96.970709 98.827679) (xy 96.952188 98.823255) (xy 96.895152 98.817567)
-					(xy 96.847122 98.820938) (xy 96.800496 98.835543) (xy 96.758645 98.868968) (xy 96.751374 98.877717)
-					(xy 96.724659 98.927953) (xy 96.713307 98.963728) (xy 96.702188 99.019519) (xy 96.700213 99.033498)
-					(xy 96.695153 99.092248) (xy 96.693762 99.151252) (xy 96.475807 99.151252) (xy 96.4758 99.150971)
-					(xy 96.475831 99.141577) (xy 96.477836 99.07868) (xy 96.482959 99.020782) (xy 96.492631 98.960735)
-					(xy 96.508382 98.900988) (xy 96.510425 98.894848) (xy 96.533509 98.837795) (xy 96.561422 98.788641)
-					(xy 96.597701 98.743696) (xy 96.627334 98.716661) (xy 96.676523 98.684272) (xy 96.7314 98.661679)
-					(xy 96.780625 98.649089) (xy 96.83737 98.640626) (xy 96.896838 98.637804)
-				)
-			)
+					(xy 97.18193 99.087211) (xy 97.302989 98.940031) (xy 96.933914 98.637804) (xy 96.798249 98.637804)
+					(xy 96.798249 99.446737) (xy 96.556412 99.446737) (xy 96.556412 99.6265) (xy 97.260295 99.6265)
+					(xy 97.260295 99.446737) (xy 97.005819 99.446737) (xy 97.005819 98.941435)
+				)
+			)

Commit message: WIP feature conf (does not compile)
Other:
- board text added: "This GND pin bears too much responsibility!"
- board text removed: "This GND pin bears too much resonsibility!"
