File: hardware/abl/controller/controller.kicad_sch (KiCad schematic)
At the start: 39 parts, among them IC1 TCA6408ARSVR, IC2 TCA6408ARSVR, IC3 VEML6040A3OG, IC4 TXB0104RUT, J1 SFW20S-2STE1LF, J2 Conn_02x05_Odd_Even, J3 Conn_02x05_Odd_Even, J4 PRT-14417, J5 Conn_02x05_Odd_Even, J6 Conn_01x10_Pin, J7 Conn_01x10_Pin, Q2 AO3401A, Q4 AO3401A, U1 INA219AxD

Commit message: Many small adjustments for the next production run.
Parts:
- J1, R4, R5: now fitted
- J2, J3: LCSC Part # C7501276 -> (none); now fitted
Changed lines of the file:
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@@
 		(in_bom yes)
 		(on_board yes)
-		(dnp yes)
+		(dnp no)
 		(fields_autoplaced yes)
 		(property "Reference" "R4"
@@
 		(in_bom yes)
 		(on_board yes)
-		(dnp yes)
+		(dnp no)
 		(property "Reference" "J3"
 			(at 235.585 53.34 0)
@@
 			)
 		)
-		(property "Description" "Generic connector, double row, 02x05, odd/even pin numbering scheme (row 1 odd numbers, row 2 even numbers), script generated (kicad-library-utils/schlib/autogen/connector/)"
+		(property "Description" ""
 			(at 227.33 52.07 0)
 			(effects
@@
 			)
 		)
-		(property "LCSC Part #" "C7501276"
+		(property "LCSC Part #" ""
 			(at 227.33 52.07 0)
 			(effects
@@
 		(in_bom yes)
 		(on_board yes)
-		(dnp yes)
+		(dnp no)
 		(property "Reference" "J2"
 			(at 200.025 53.34 0)
@@
 			)
 		)
-		(property "Description" "Generic connector, double row, 02x05, odd/even pin numbering scheme (row 1 odd numbers, row 2 even numbers), script generated (kicad-library-utils/schlib/autogen/connector/)"
+		(property "Description" ""
 			(at 191.135 52.07 0)
 			(effects
@@
 			)
 		)
-		(property "LCSC Part #" "C7501276"
+		(property "LCSC Part #" ""
 			(at 191.135 52.07 0)
 			(effects
@@
 		(in_bom yes)
 		(on_board yes)
-		(dnp yes)
+		(dnp no)
 		(property "Reference" "R5"
 			(at 98.425 175.26 0)
@@
 		(in_bom yes)
 		(on_board yes)
-		(dnp yes)
+		(dnp no)
 		(property "Reference" "J1"
 			(at 42.545 86.36 90)

Commit message: WIP feature conf (does not compile)
Parts:
- J1: LCSC Part # C5407823 -> C3168412
Changed lines of the file:
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@@
 	(title_block
 		(title "besteLampe! ABL Controller Module")
-		(date "2024-11-15")
-		(rev "1.1")
+		(date "2024-12-01")
+		(rev "1.2")
 		(comment 1 "See  https://beste-lampe.de for the source and more information")
 		(comment 2 "This source describes Open Hardware and is licensed under the CERN-OHL-S v2.")
@@
 			)
 		)
-		(property "LCSC Part #" "C5407823"
+		(property "LCSC Part #" "C3168412"
 			(at 50.8 75.565 0)
 			(effects
