File: hardware/abl/LED_Module_E/LED_Module_E.kicad_pcb (KiCad board)
At the start: 4 copper layers, 140.8 x 26 mm, 97 parts, among them J1 SFW20S-2STE1LF, J3 009159008603906, K1 Conn_01x01, K10 Conn_01x01, K11 Conn_01x01, K12 Conn_01x01, K13 Conn_01x01, K14 Conn_01x01, K15 Conn_01x01, K16 Conn_01x01, K17 Conn_01x01, K18 Conn_01x01, K19 Conn_01x01, K2 Conn_01x01, K3 Conn_01x01, K4 Conn_01x01, K5 Conn_01x01, K6 Conn_01x01, K7 Conn_01x01, K8 Conn_01x01, K9 Conn_01x01, Q1 Si3456DDV, Q11 Si3456DDV, Q12 Si3456DDV, Q2 Si3456DDV, Q3 Si3456DDV, Q4 Si3456DDV, Q5 Si3456DDV, Q6 Si3456DDV, Q7 Si3456DDV, Q8 Si3456DDV, U2 74HC245, U3 24AA025E48T-I/OT, U4 74LVC1G32

Commit message: WUP LED Module E
Parts:
- TP10, TP11, TP12, TP13, TP14, TP5, TP6, TP7, TP8, TP9: footprint TestPoint:TestPoint_Pad_D1.0mm -> TestPoint:TestPoint_THTPad_D1.0mm_Drill0.5mm
- moved TP9 77.1 mm to (173.2, 66.0), turned to 90 degrees
- moved TP10 71.2 mm to (166.2, 63.8), turned to 90 degrees
- moved TP11 65.0 mm to (158.7, 60.8), turned to 90 degrees
- moved TP12 21.6 mm to (113.0, 58.2)
- moved TP7 17.2 mm to (90.8, 74.7)
- moved TP13 16.3 mm to (106.2, 59.8)
- moved H8 11.8 mm to (103.2, 63.5)
- moved TP14 8.56 mm to (98.5, 65.5)
- moved TP8 7.97 mm to (94.4, 67.9), turned to 135 degrees
- moved R10 6.31 mm to (96.0, 80.0), turned to 180 degrees
- moved Q11 5.41 mm to (94.3, 75.2), turned to -90 degrees
- moved R17 4.83 mm to (115.0, 67.2)
- moved R7 4.83 mm to (112.0, 64.2)
- moved Q7 4.49 mm to (108.5, 62.2)
- moved R16 4.46 mm to (121.7, 66.0), turned to 120 degrees
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Routing:
- net Net-(Q12-G): track 125.6 -> 75.0 mm, vias 2 -> 1
- net Net-(Q3-G): track 108.9 -> 73.9 mm, vias 0 -> 1
- net Net-(Q1-G): track 126.9 -> 94.9 mm, vias 2 -> 1
- net GND: track 54.0 -> 26.8 mm, vias 196 -> 94
- net Net-(Q4-G): track 101.8 -> 84.7 mm, vias 0 -> 1
- net /ALERT: track 98.8 -> 84.3 mm, vias 3 -> 1
- net Net-(U2-CE): track 16.7 -> 12.9 mm
- net Net-(R19-Pad2): track 1.99 -> 0.00 mm, vias 15 -> 0
- net Net-(R18-Pad2): track 1.99 -> 0.00 mm, vias 10 -> 0
- net Net-(R17-Pad2): track 1.99 -> 0.00 mm, vias 9 -> 0
- net Net-(R16-Pad2): track 1.99 -> 0.00 mm, vias 9 -> 0
- net Net-(R10-Pad1): track 1.99 -> 0.00 mm, vias 15 -> 0
- net Net-(Q6-G): track 44.4 -> 45.8 mm, vias 0 -> 1
- net /SCL: track 72.1 -> 73.3 mm
- net Net-(Q8-G): track 27.1 -> 28.3 mm, vias 0 -> 1
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- added copper zone on In1.Cu, net +4V
- removed copper zone on B.Cu, net Net-(R1-Pad1)
- removed copper zone on B.Cu, net Net-(R10-Pad1)
- removed copper zone on B.Cu, net Net-(R12-Pad2)
- removed copper zone on B.Cu, net Net-(R13-Pad2)
- removed copper zone on B.Cu, net Net-(R14-Pad2)
- removed copper zone on B.Cu, net Net-(R15-Pad2)
- removed copper zone on B.Cu, net Net-(R16-Pad2)
- removed copper zone on B.Cu, net Net-(R17-Pad2)
- removed copper zone on B.Cu, net Net-(R18-Pad2)
- removed copper zone on B.Cu, net Net-(R19-Pad2)
